File: KICAD/ASGARD.kicad_pcb (KiCad board)
At the start: 4 copper layers, 50 x 150 mm, 157 parts, among them J1 BATT_TERM, J12 LED_OUT, J13 UART1, J14 UART2, J17 SMA, J18 I2C0, J2 ARMING/GPIO, J21 I2C1/UART4, J3 PYRO_TERM_A, J4 PYRO_TERM_B, J5 POWER_OUT, J6 SWITCH_TERM, J7 SPI0, J8 SPI1, J9 CAN_OUT, M1 FIN_X+, M2 FIN_X-, M3 FIN_Y+, M4 FIN_Y-, M5 TVC_X, M6 TVC_Y, Q1 PY_3A_MOSFET, Q10 VCC_SERVO_ARM_MOSFET, Q2 PY_2A_MOSFET, Q3 PY_1A_MOSFET, Q4 PY_3B_MOSFET, Q5 PY_2B_MOSFET, Q6 PY_1B_MOSFET, Q7 PYRO_ARM_MOSFET, Q8 PYRO_ARM_TRANS, Q9 5V_SERVO_ARM_MOSFET, U1 Teensy4.1, U10 BMI270, U11 MS5607-02BA, U2 INA226, U3 LMR51460SQDRRRQ1, U4 BMI088, U5 H3LIS331DLTR, U6 BMP581, U7 MMC5983MA, U8 MAX-M10S, U9 TCAN332G

Commit message: gnss complete. only sensors left
Parts:
- removed C22: 47pF, Capacitor_SMD:C_0603_1608Metric
- C17, C20, C25: value 10uF 25V -> 10uF
- moved R80 32.5 mm to (70.0, 42.0), turned to 0 degrees
- moved R77 30.9 mm to (65.2, 26.5), turned to 180 degrees
- moved D25 29.8 mm to (70.0, 39.5), turned to 180 degrees
- moved C18 29.7 mm to (70.0, 34.5)
- moved C20 29.7 mm to (70.0, 37.0)
- moved U8 19.3 mm to (60.5, 33.3), turned to 180 degrees
- moved R53 8.46 mm to (51.5, 37.8), turned to 180 degrees
- moved C21 6.03 mm to (47.5, 37.8)
- moved L2 5.33 mm to (51.5, 35.2)
Connections:
- U8 pad 11: Net-(U8-RF_IN) -> Net-(J17-In)
Routing:
- net GND: track 299.7 -> 918.3 mm, vias 15 -> 104
- net +3.3V: track 396.9 -> 428.6 mm, vias 5 -> 8
- net VCC: track 202.7 -> 183.5 mm
- net /BYPASS: track 65.2 -> 81.9 mm
- net /VCC_SERVO_MOSFET: track 29.9 -> 35.4 mm
- net Net-(U8-RF_IN): track 4.25 -> 0.00 mm
- net TIMEPULSE: track 2.77 -> 6.85 mm
- net SCL0: track 178.4 -> 174.7 mm
- net FIN_X+_PWM: track 78.9 -> 81.4 mm
- net TX1: track 25.3 -> 23.4 mm
- net RX1: track 24.5 -> 22.6 mm
- net SDA0: track 161.9 -> 163.6 mm
- net PYRO_3B: track 11.2 -> 9.75 mm
- net PYRO_3A: track 26.0 -> 24.6 mm
- net PYRO_2B: track 14.1 -> 12.7 mm
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- added copper zone on B.Cu, net GND
- added copper zone on F.Cu, net GND
- added copper zone on In1.Cu, net GND
- added copper zone on In2.Cu, net GND
Other:
- board text added: "Add more vias around the outside of bias tee and max-m10s"

Commit message: completed routing
Parts:
- moved C14 62.3 mm to (40.0, 51.2)
- moved C25 61.9 mm to (40.0, 53.8), turned to 180 degrees
- moved C24 56.6 mm to (40.0, 43.8)
- moved C23 56.4 mm to (40.0, 41.2), turned to 180 degrees
- moved C13 56.1 mm to (40.0, 48.8)
- moved C12 56.0 mm to (40.0, 46.2), turned to 180 degrees
- moved U5 53.4 mm to (45.0, 52.5)
- moved U7 53.1 mm to (55.0, 42.5)
- moved C15 52.8 mm to (60.0, 52.5), turned to 180 degrees
- moved C16 52.6 mm to (60.0, 41.2)
- moved C17 52.3 mm to (60.0, 43.8)
- moved U6 52.1 mm to (55.0, 47.5)
- moved U11 51.8 mm to (55.0, 52.5)
- moved C11 51.4 mm to (60.0, 47.5), turned to 180 degrees
- moved U10 46.9 mm to (45.0, 42.5)
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Connections:
- R78 pad 1: CS_L-IMU -> CS_L-BARO
- R79 pad 1: CS_M-IMU_ACCL -> CS_MAG
- R81 pad 1: CS_M-IMU_GYRO -> CS_L-IMU
- R82 pad 1: CS_H-ACCL -> CS_M-IMU_GYRO
- R83 pad 1: CS_L-BARO -> CS_M-IMU_ACCL
- R84 pad 1: CS_H-BARO -> CS_H-ACCL
- R85 pad 1: CS_MAG -> CS_H-BARO
- U1 pad 26: CS_H-BARO -> CS_H-ACCL
- U1 pad 27: CS_L-BARO -> CS_M-IMU_ACCL
- U1 pad 28: CS_H-ACCL -> CS_M-IMU_GYRO
- U1 pad 29: CS_M-IMU_GYRO -> CS_L-IMU
- U1 pad 30: CS_M-IMU_ACCL -> CS_MAG
- U1 pad 32: CS_L-IMU -> CS_L-BARO
- U1 pad 33: CS_MAG -> CS_H-BARO
Routing:
- net GND: track 918.3 -> 1030.6 mm
- net +3.3V: track 428.6 -> 533.4 mm, vias 8 -> 15
- net POCI0: track 38.9 -> 115.5 mm, vias 0 -> 5
- net PICO1: track 49.5 -> 119.4 mm, vias 0 -> 2
- net SCK1: track 52.4 -> 117.6 mm, vias 0 -> 3
- net PICO0: track 35.9 -> 98.7 mm, vias 0 -> 2
- net POCI1: track 50.7 -> 113.4 mm, vias 0 -> 6
- net SCK0: track 39.7 -> 101.3 mm, vias 0 -> 8
- net CS_L-IMU: track 50.0 -> 87.2 mm, vias 0 -> 2
- net CS_MAG: track 47.3 -> 82.0 mm, vias 0 -> 2
- net CS_M-IMU_ACCL: track 55.8 -> 84.0 mm, vias 0 -> 2
- net CS_M-IMU_GYRO: track 58.5 -> 86.5 mm, vias 0 -> 2
- net CS_H-ACCL: track 61.2 -> 79.9 mm, vias 0 -> 2
- net CS_L-BARO: track 63.9 -> 71.4 mm, vias 0 -> 2
- net CS_H-BARO: track 66.6 -> 62.3 mm, vias 0 -> 2
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Other:
- board text removed: "I2C1 PULL UP"
