File: KICAD/ASGARD.kicad_sch (KiCad schematic)
At the start: 157 parts, among them J1 BATT_TERM, J12 LED_OUT, J13 UART1, J14 UART2, J17 SMA, J18 I2C0, J2 ARMING/GPIO, J21 I2C1/UART4, J3 PYRO_TERM_A, J4 PYRO_TERM_B, J5 POWER_OUT, J6 SWITCH_TERM, J7 SPI0, J8 SPI1, J9 CAN_OUT, M1 FIN_X+, M2 FIN_X-, M3 FIN_Y+, M4 FIN_Y-, M5 TVC_X, M6 TVC_Y, Q1 PY_3A_MOSFET, Q10 VCC_SERVO_ARM_MOSFET, Q2 PY_2A_MOSFET, Q3 PY_1A_MOSFET, Q4 PY_3B_MOSFET, Q5 PY_2B_MOSFET, Q6 PY_1B_MOSFET, Q7 PYRO_ARM_MOSFET, Q8 PYRO_ARM_TRANS, Q9 5V_SERVO_ARM_MOSFET, U1 Teensy4.1, U10 BMI270, U11 MS5607-02BA, U2 INA226, U3 LMR51460SQDRRRQ1, U4 BMI088, U5 H3LIS331DLTR, U6 BMP581, U7 MMC5983MA, U8 MAX-M10S, U9 TCAN332G

Commit message: gnss complete. only sensors left
Parts:
- removed C22: 47pF, Capacitor_SMD:C_0603_1608Metric, symbol Device:C
- C17, C20, C25: value 10uF 25V -> 10uF
Connections:
- net at U8.11 (RF_IN): now also J17.1 (In), L2.2
Other:
- moved on the sheet: C14, C25
Changed lines of the file:
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@@
 	)
 	(junction
-		(at 342.9 119.38)
-		(diameter 0)
-		(color 0 0 0 0)
-	)
-	(junction
 		(at 24.13 19.05)
 		(diameter 0)
@@
 	)
 	(junction
-		(at 123.19 123.19)
+		(at 328.93 104.14)
 		(diameter 0)
 		(color 0 0 0 0)
 	)
 	(junction
-		(at 220.98 129.54)
+		(at 123.19 123.19)
 		(diameter 0)
 		(color 0 0 0 0)
 	)
 	(junction
-		(at 342.9 104.14)
+		(at 220.98 129.54)
 		(diameter 0)
 		(color 0 0 0 0)
@@
 	)
 	(junction
+		(at 328.93 119.38)
+		(diameter 0)
+		(color 0 0 0 0)
+	)
+	(junction
 		(at 34.29 140.97)
 		(diameter 0)
@@
 	)
 	(junction
+		(at 342.9 119.38)
+		(diameter 0)
+		(color 0 0 0 0)
+	)
+	(junction
 		(at 243.84 139.7)
 		(diameter 0)
@@
 	)
 	(junction
+		(at 342.9 104.14)
+		(diameter 0)
+		(color 0 0 0 0)
+	)
+	(junction
 		(at 383.54 78.74)
 		(diameter 0)
@@
 	)
 	(junction
-		(at 328.93 104.14)
-		(diameter 0)
-		(color 0 0 0 0)
-	)
-	(junction
 		(at 123.19 34.29)
 		(diameter 0)
@@
 	)
 	(junction
-		(at 328.93 119.38)
-		(diameter 0)
-		(color 0 0 0 0)
-	)
-	(junction
 		(at 16.51 109.22)
 		(diameter 0)
@@
 	(wire
 		(pts
-			(xy 342.9 105.41) (xy 342.9 104.14)
+			(xy 342.9 107.95) (xy 342.9 104.14)
 		)
 		(stroke
@@
 	(wire
 		(pts
-			(xy 224.79 190.5) (xy 222.25 190.5)
+			(xy 222.25 190.5) (xy 238.76 190.5)
 		)
 		(stroke
@@
 	(wire
 		(pts
-			(xy 342.9 113.03) (xy 342.9 119.38)
+			(xy 342.9 115.57) (xy 342.9 119.38)
 		)
 		(stroke
@@
 	(wire
 		(pts
-			(xy 328.93 118.11) (xy 328.93 119.38)
+			(xy 328.93 115.57) (xy 328.93 119.38)
 		)
 		(stroke
@@
 	(wire
 		(pts
-			(xy 238.76 190.5) (xy 232.41 190.5)
-		)
-		(stroke
-			(width 0)
-			(type default)
-		)
-	)
-	(wire
-		(pts
 			(xy 115.57 105.41) (xy 115.57 104.14)
 		)
@@
 	(wire
 		(pts
-			(xy 328.93 104.14) (xy 328.93 110.49)
+			(xy 328.93 104.14) (xy 328.93 107.95)
 		)
 		(stroke
@@
 			)
 		)
-		(property "Value" "10uF 25V"
+		(property "Value" "10uF"
 			(at 176.53 181.61 90)
 			(show_name no)
@@
 			)
 		)
-		(property "Value" "10uF 25V"
+		(property "Value" "10uF"
 			(at 339.09 217.1699 0)
 			(show_name no)
@@
 	(symbol
 		(lib_id "Device:C")
-		(at 342.9 109.22 180)
+		(at 342.9 111.76 180)
 		(unit 1)
 		(body_style 1)
@@
 		(dnp no)
 		(property "Reference" "C14"
-			(at 346.71 107.9499 0)
+			(at 346.71 110.4899 0)
 			(show_name no)
 			(do_not_autoplace no)
@@
 		)
 		(property "Value" "100nF"
-			(at 345.948 110.49 0)
+			(at 345.948 113.03 0)
 			(show_name no)
 			(do_not_autoplace no)
@@
 		)
 		(property "Footprint" "Capacitor_SMD:C_0603_1608Metric"
-			(at 341.9348 105.41 0)
+			(at 341.9348 107.95 0)
 			(hide yes)
 			(show_name no)
@@
 		)
 		(property "Datasheet" ""
-			(at 342.9 109.22 0)
+			(at 342.9 111.76 0)
 			(hide yes)
 			(show_name no)
@@
 		)
 		(property "Description" "Unpolarized capacitor"
-			(at 342.9 109.22 0)
+			(at 342.9 111.76 0)
 			(hide yes)
 			(show_name no)
@@
 	)
 	(symbol
-		(lib_id "Device:C")
-		(at 228.6 190.5 90)
-		(unit 1)
-		(body_style 1)
-		(exclude_from_sim no)
-		(in_bom yes)
-		(on_board yes)
-		(in_pos_files yes)
-		(dnp no)
-		(fields_autoplaced yes)
-		(property "Reference" "C22"
-			(at 228.6 182.88 90)
-			(show_name no)
-			(do_not_autoplace no)
-			(effects
-				(font
-					(size 1.27 1.27)
-				)
-			)
-		)
-		(property "Value" "47pF"
-			(at 228.6 185.42 90)
-			(show_name no)
-			(do_not_autoplace no)
-			(effects
-				(font
-					(size 1.27 1.27)
-				)
-			)
-		)
-		(property "Footprint" "Capacitor_SMD:C_0603_1608Metric"
-			(at 232.41 189.5348 0)
-			(hide yes)
-			(show_name no)
-			(do_not_autoplace no)
-			(effects
-				(font
-					(size 1.27 1.27)
-				)
-			)
-		)
-		(property "Datasheet" ""
-			(at 228.6 190.5 0)
-			(hide yes)
-			(show_name no)
-			(do_not_autoplace no)
-			(effects
-				(font
-					(size 1.27 1.27)
-				)
-			)
-		)
-		(property "Description" "Unpolarized capacitor"
-			(at 228.6 190.5 0)
-			(hide yes)
-			(show_name no)
-			(do_not_autoplace no)
-			(effects
-				(font
-					(size 1.27 1.27)
-				)
-			)
-		)
-		(pin "2"
-		)
-		(pin "1"
-		)
-		(instances
-			(project "ASGARD"
-				(path "/1109dbdb-412c-44ab-a4bd-b3242fa9b951"
-					(reference "C22")
-					(unit 1)
-				)
-			)
-		)
-	)
-	(symbol
 		(lib_id "Device:R_US")
 		(at 393.7 190.5 90)
@@
 	(symbol
 		(lib_id "Device:C")
-		(at 328.93 114.3 0)
+		(at 328.93 111.76 0)
 		(unit 1)
 		(body_style 1)
@@
 		(fields_autoplaced yes)
 		(property "Reference" "C25"
-			(at 332.74 113.0299 0)
+			(at 332.74 110.4899 0)
 			(show_name no)
 			(do_not_autoplace no)
@@
 			)
 		)
-		(property "Value" "10uF 25V"
-			(at 332.74 115.5699 0)
+		(property "Value" "10uF"
+			(at 332.74 113.0299 0)
 			(show_name no)
 			(do_not_autoplace no)
@@
 		)
 		(property "Footprint" "Capacitor_SMD:C_0603_1608Metric"
-			(at 329.8952 118.11 0)
+			(at 329.8952 115.57 0)
 			(hide yes)
 			(show_name no)
@@
 		)
 		(property "Datasheet" ""
-			(at 328.93 114.3 0)
+			(at 328.93 111.76 0)
 			(hide yes)
 			(show_name no)
@@
 		)
 		(property "Description" "Unpolarized capacitor"
-			(at 328.93 114.3 0)
+			(at 328.93 111.76 0)
 			(hide yes)
 			(show_name no)

Commit message: completed routing
Connections:
- net CS_H-ACCL: now also R84.1, U1.26 (34_RX8); no longer R82.1, U1.28 (36_CS)
- net CS_H-BARO: now also R85.1, U1.33 (41_A17); no longer R84.1, U1.26 (34_RX8)
- net CS_L-BARO: now also R78.1, U1.32 (40_A16); no longer R83.1, U1.27 (35_TX8)
- net CS_L-IMU: now also R81.1, U1.29 (37_CS); no longer R78.1, U1.32 (40_A16)
- net CS_M-IMU_ACCL: now also R83.1, U1.27 (35_TX8); no longer R79.1, U1.30 (38_CS1_IN1)
- net CS_M-IMU_GYRO: now also R82.1, U1.28 (36_CS); no longer R81.1, U1.29 (37_CS)
- net CS_MAG: now also R79.1, U1.30 (38_CS1_IN1); no longer R85.1, U1.33 (41_A17)
